File: ESPMDIR/ESPMDIR.brd (EAGLE design)
At the start: 100 x 83.8 mm, 40 parts, among them IC1 TSOP34830, IC2 LM1117MP-3.3, IC3 LM1117MP-5.0, X2 2N7002, X3 2N7002, X4 2N7002

Commit message: 11092017
Parts:
- removed R16: 10k, rcl:R0805
- moved C3 7.10 mm to (47.0, 48.3), turned to 0 degrees
- moved C2 3.42 mm to (55.9, 40.6)
- moved SJ1 2.01 mm to (27.9, 41.9), turned to 90.5 degrees
- moved IC2 1.42 mm to (48.9, 42.5), turned to 180 degrees
Connections:
- removed net N$19 (its old number): C5.1, D5.C, IC3.3
- removed net N$34: R15.1, R16.1, U$1.CH_PD
- new net N$29: C5.1, D5.C, IC2.3, IC3.3
- net N$10: no longer IC2.3
- net N$5: now also R15.1, U$1.CH_PD; no longer R16.2
Routing:
- net N$29: track 0.00 -> 26.2 mm
- net N$19: track 181.5 -> 200.0 mm
- net N$19 (its old number): track 18.5 -> 0.00 mm
- net N$26: track 0.00 -> 18.2 mm, vias 0 -> 1
- net N$34: track 16.9 -> 0.00 mm
- net N$30: track 0.00 -> 5.71 mm
- net N$5: track 72.6 -> 78.0 mm, vias 2 -> 1
- net N$10: track 78.9 -> 83.0 mm
- net N$12: track 81.2 -> 83.2 mm
Other:
- board size 100 x 83.8 mm -> 57.8 x 47.6 mm
- board text added: "09.2017"
- board text added: "Гамаев Влад"
