File: ESPMDIR/ESPMDIR.sch (EAGLE design)
At the start: 40 parts, among them IC1 TSOP34830, IC2 LM1117MP-3.3, IC3 LM1117MP-5.0, X2 2N7002, X3 2N7002, X4 2N7002

Commit message: 11092017
Parts:
- removed R16: 10k, rcl:R-EU_R0805
Connections:
- removed net N$19 (its old number): C5.1, D5.C, IC3.IN
- removed net N$34: R15.1, R16.1, U$1.CH_PD
- new net N$29: C5.1, D5.C, IC2.IN, IC3.IN
- net N$10: no longer IC2.IN
- net N$5: now also R15.1, U$1.CH_PD; no longer R16.2
Other:
- moved on the sheet: C2
Changed lines of the file:
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@@
 <part name="JP4" library="pinhead" deviceset="PINHD-1X2" device=""/>
 <part name="GND18" library="supply1" deviceset="GND" device=""/>
-<part name="R16" library="rcl" deviceset="R-EU_" device="R0805" value="10k"/>
 <part name="R17" library="rcl" deviceset="R-EU_" device="R0805" value="10k"/>
 <part name="GND19" library="supply1" deviceset="GND" device=""/>
@@
 <instance part="R10" gate="G$1" x="83.82" y="5.08" rot="R90"/>
 <instance part="C1" gate="G$1" x="38.1" y="30.48"/>
-<instance part="C2" gate="G$1" x="63.5" y="38.1"/>
+<instance part="C2" gate="G$1" x="60.96" y="27.94"/>
 <instance part="C3" gate="G$1" x="93.98" y="38.1"/>
 <instance part="R11" gate="G$1" x="88.9" y="5.08" rot="R90"/>
@@
 <instance part="GND3" gate="1" x="101.6" y="48.26"/>
 <instance part="GND4" gate="1" x="129.54" y="20.32"/>
-<instance part="GND5" gate="1" x="63.5" y="27.94"/>
+<instance part="GND5" gate="1" x="60.96" y="20.32"/>
 <instance part="GND6" gate="1" x="93.98" y="27.94"/>
 <instance part="SJ1" gate="G$1" x="66.04" y="10.16" rot="R180"/>
@@
 <instance part="JP4" gate="G$1" x="-5.08" y="-17.78"/>
 <instance part="GND18" gate="1" x="2.54" y="-22.86"/>
-<instance part="R16" gate="G$1" x="60.96" y="66.04" rot="R270"/>
 <instance part="R17" gate="G$1" x="109.22" y="55.88" rot="R270"/>
 <instance part="GND19" gate="1" x="109.22" y="48.26"/>
@@
 <junction x="68.58" y="58.42"/>
 <pinref part="C4" gate="G$1" pin="1"/>
-<pinref part="R16" gate="G$1" pin="2"/>
 <wire x1="60.96" y1="60.96" x2="60.96" y2="58.42" width="0.1524" layer="91"/>
 <wire x1="63.5" y1="60.96" x2="60.96" y2="60.96" width="0.1524" layer="91"/>
+<pinref part="R15" gate="G$1" pin="1"/>
+<pinref part="U$1" gate="G$1" pin="CH_PD"/>
+<wire x1="68.58" y1="71.12" x2="60.96" y2="71.12" width="0.1524" layer="91"/>
+<wire x1="60.96" y1="71.12" x2="53.34" y2="71.12" width="0.1524" layer="91"/>
+<wire x1="60.96" y1="60.96" x2="60.96" y2="71.12" width="0.1524" layer="91"/>
 <junction x="60.96" y="60.96"/>
+<junction x="60.96" y="71.12"/>
 </segment>
 </net>
@@
 </segment>
 </net>
-<net name="N$26" class="0">
+<net name="N$19" class="0">
 <segment>
 <pinref part="IC1" gate="G$1" pin="GND"/>
@@
 <pinref part="C2" gate="G$1" pin="2"/>
 <pinref part="GND5" gate="1" pin="GND"/>
-<wire x1="63.5" y1="30.48" x2="63.5" y2="33.02" width="0.1524" layer="91"/>
 </segment>
 <segment>
@@
 <pinref part="SJ1" gate="G$1" pin="1"/>
 <wire x1="66.04" y1="5.08" x2="55.88" y2="5.08" width="0.1524" layer="91"/>
-<pinref part="IC2" gate="G$1" pin="IN"/>
-<pinref part="C2" gate="G$1" pin="1"/>
-<wire x1="68.58" y1="40.64" x2="63.5" y2="40.64" width="0.1524" layer="91"/>
-<wire x1="63.5" y1="40.64" x2="55.88" y2="40.64" width="0.1524" layer="91"/>
-<junction x="63.5" y="40.64"/>
 <wire x1="55.88" y1="5.08" x2="55.88" y2="35.56" width="0.1524" layer="91"/>
 <pinref part="R14" gate="G$1" pin="1"/>
-<wire x1="55.88" y1="35.56" x2="55.88" y2="40.64" width="0.1524" layer="91"/>
 <wire x1="50.8" y1="35.56" x2="55.88" y2="35.56" width="0.1524" layer="91"/>
-<junction x="55.88" y="35.56"/>
 <pinref part="IC3" gate="G$1" pin="OUT"/>
 <wire x1="38.1" y1="-10.16" x2="43.18" y2="-10.16" width="0.1524" layer="91"/>
@@
 <wire x1="43.18" y1="5.08" x2="55.88" y2="5.08" width="0.1524" layer="91"/>
 <junction x="55.88" y="5.08"/>
+<pinref part="C2" gate="G$1" pin="1"/>
+<wire x1="60.96" y1="30.48" x2="60.96" y2="35.56" width="0.1524" layer="91"/>
+<wire x1="60.96" y1="35.56" x2="55.88" y2="35.56" width="0.1524" layer="91"/>
+<junction x="55.88" y="35.56"/>
 </segment>
 </net>
@@
 </segment>
 </net>
-<net name="N$19" class="0">
-<segment>
-<pinref part="IC3" gate="G$1" pin="IN"/>
-<pinref part="D5" gate="G$1" pin="C"/>
-<wire x1="22.86" y1="-10.16" x2="17.78" y2="-10.16" width="0.1524" layer="91"/>
-<pinref part="C5" gate="G$1" pin="1"/>
-<wire x1="17.78" y1="-10.16" x2="7.62" y2="-10.16" width="0.1524" layer="91"/>
-<wire x1="17.78" y1="-12.7" x2="17.78" y2="-10.16" width="0.1524" layer="91"/>
-<junction x="17.78" y="-10.16"/>
-</segment>
-</net>
 <net name="N$33" class="0">
 <segment>
@@
 </segment>
 </net>
-<net name="N$34" class="0">
-<segment>
-<pinref part="R15" gate="G$1" pin="1"/>
-<pinref part="U$1" gate="G$1" pin="CH_PD"/>
-<wire x1="68.58" y1="71.12" x2="60.96" y2="71.12" width="0.1524" layer="91"/>
-<pinref part="R16" gate="G$1" pin="1"/>
-<wire x1="60.96" y1="71.12" x2="53.34" y2="71.12" width="0.1524" layer="91"/>
-<junction x="60.96" y="71.12"/>
-</segment>
-</net>
+<net name="N$29" class="0">
+<segment>
+<wire x1="50.8" y1="40.64" x2="50.8" y2="10.16" width="0.1524" layer="91"/>
+<wire x1="50.8" y1="10.16" x2="38.1" y2="10.16" width="0.1524" layer="91"/>
+<wire x1="38.1" y1="10.16" x2="38.1" y2="0" width="0.1524" layer="91"/>
+<pinref part="IC3" gate="G$1" pin="IN"/>
+<pinref part="D5" gate="G$1" pin="C"/>
+<wire x1="22.86" y1="-10.16" x2="17.78" y2="-10.16" width="0.1524" layer="91"/>
+<pinref part="C5" gate="G$1" pin="1"/>
+<wire x1="17.78" y1="-10.16" x2="7.62" y2="-10.16" width="0.1524" layer="91"/>
+<wire x1="17.78" y1="-12.7" x2="17.78" y2="-10.16" width="0.1524" layer="91"/>
+<junction x="17.78" y="-10.16"/>
+<wire x1="38.1" y1="0" x2="17.78" y2="0" width="0.1524" layer="91"/>
+<wire x1="17.78" y1="0" x2="17.78" y2="-10.16" width="0.1524" layer="91"/>
+<pinref part="IC2" gate="G$1" pin="IN"/>
+<wire x1="50.8" y1="40.64" x2="68.58" y2="40.64" width="0.1524" layer="91"/>
+</segment>
+</net>
